File: schematics/auxiliary/auxiliary.kicad_sch (KiCad schematic)
At the start: 4 parts, among them J1 Conn_01x04_Male, SW1 SW_Push, SW2 SW_Push, SW3 SW_Push

Commit message: cleanup, added net labels
Parts:
- J1: value Conn_01x04_Male -> CONN
Connections:
- net DOWN: now reaches J1.2 (Pin_2), SW2.1
- net GND: now reaches J1.4 (Pin_4), SW1.2, SW2.2, SW3.2
- net UP: now reaches J1.1 (Pin_1), SW1.1
- net SET: now reaches J1.3 (Pin_3), SW3.1
Changed lines of the file:
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@@
+    (stroke (width 0) (type default) (color 0 0 0 0))
+  )
+  (wire (pts (xy 41.91 49.53) (xy 36.83 49.53))
     (stroke (width 0) (type default) (color 0 0 0 0))
   )
@@
     (stroke (width 0) (type default) (color 0 0 0 0))
   )
-  (wire (pts (xy 36.83 64.77) (xy 36.83 49.53))
+  (wire (pts (xy 41.91 64.77) (xy 41.91 49.53))
     (stroke (width 0) (type default) (color 0 0 0 0))
   )
@@
     (stroke (width 0) (type default) (color 0 0 0 0))
   )
-  (wire (pts (xy 64.77 64.77) (xy 36.83 64.77))
+  (wire (pts (xy 64.77 64.77) (xy 41.91 64.77))
     (stroke (width 0) (type default) (color 0 0 0 0))
   )
@@
   (wire (pts (xy 60.96 62.23) (xy 64.77 62.23))
     (stroke (width 0) (type default) (color 0 0 0 0))
+  )
+  (label "GND" (at 36.83 49.53 0)
+    (effects (font (size 1.27 1.27)) (justify left bottom))
+  )
+  (label "DOWN" (at 36.83 44.45 0)
+    (effects (font (size 1.27 1.27)) (justify left bottom))
+  )
+  (label "UP" (at 36.83 41.91 0)
+    (effects (font (size 1.27 1.27)) (justify left bottom))
+  )
+  (label "SET" (at 36.83 46.99 0)
+    (effects (font (size 1.27 1.27)) (justify left bottom))
   )
   (symbol (lib_id "Switch:SW_Push") (at 55.88 52.07 0) (unit 1)
@@
     (in_bom yes) (on_board yes) (fields_autoplaced)
     (property "Reference" "J1" (id 0) (at 32.385 36.83 0))
-    (property "Value" "Conn_01x04_Male" (id 1) (at 32.385 39.37 0))
+    (property "Value" "CONN" (id 1) (at 32.385 39.37 0))
     (property "Footprint" "Connector_PinHeader_2.54mm:PinHeader_1x04_P2.54mm_Horizontal" (id 2) (at 31.75 44.45 0)
       (effects (font (size 1.27 1.27)) hide)
@@
   (symbol_instances
     (path "/47a62489-3f12-4047-a40d-0aa970bb624a"
-      (reference "J1") (unit 1) (value "Conn_01x04_Male") (footprint "Connector_PinHeader_2.54mm:PinHeader_1x04_P2.54mm_Horizontal")
+      (reference "J1") (unit 1) (value "CONN") (footprint "Connector_PinHeader_2.54mm:PinHeader_1x04_P2.54mm_Horizontal")
     )
     (path "/9ae8bfcc-ca84-423d-8f07-086e22fb905f"
