File: schematics/mainboard/mainboard.kicad_pcb (KiCad board)
At the start: 2 copper layers, 94.6 x 55.9 mm, 33 parts, among them J1 Nav Pin, J2 LCD I2C, J3 Serial ESP, J4 RTC DS1307, J5 PWR, J6 Temp DS18B20, J7 Serial ATMega, J8 Relay Module, U1 ESP-12E, U2 ATmega328-P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

Commit message: minor fix schematics
Parts:
- removed REF** (x4): MountingHole_3.2mm_M3, MountingHole:MountingHole_3.2mm_M3
- C1, C2, C3, C4: footprint Capacitor_THT:C_Disc_D4.3mm_W1.9mm_P5.00mm -> Capacitor_THT:C_Disc_D4.7mm_W2.5mm_P5.00mm
- J5: footprint TerminalBlock_4Ucon:TerminalBlock_4Ucon_1x03_P3.50mm_Horizontal -> TerminalBlock:TerminalBlock_bornier-3_P5.08mm
- moved J5 1.80 mm to (74.9, 68.6)
- renumbered RST to SW1, FLASH to SW2, RST_AM to SW3
Connections:
- net Net-(J1-Pad1) renamed /UP
- net Net-(J1-Pad2) renamed /DOWN
- net Net-(J1-Pad3) renamed /SET
- net Net-(J2-Pad3) renamed /SDA
- net Net-(J2-Pad4) renamed /SCL
- net Net-(J3-Pad1) renamed /TX_ESP
- net Net-(J3-Pad2) renamed /RX_ESP
- net Net-(J6-Pad2) renamed /DQ
- net Net-(J7-Pad1) renamed /TX_ATMega
- net Net-(J7-Pad2) renamed /RX_ATMega
- net Net-(J8-Pad1) renamed /CH1
- net Net-(J8-Pad2) renamed /CH2
- net Net-(J8-Pad3) renamed /CH3
- J4 pad 1: unconnected-(J4-Pad1) -> /OS
Routing:
- net +5V: track 104.4 -> 102.7 mm
- net GND: track 418.9 -> 419.8 mm
- net +3.3V: track 147.5 -> 146.7 mm
